File: hardware/vgagenerator.kicad_pcb (KiCad board)
At the start: 2 copper layers, 90 parts, among them J1 VGA1, J2 VGA2, J3 VGA3, J4 VGA4, U1 Pico, U2 74HC374, U3 74HC374, U4 74HC374, U5 74HC374, U6 74HC374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

Commit message: Updated schematics
Parts:
- added C9: 10uF x 10V, Capacitor_THT:C_Radial_D6.3mm_H11.0mm_P2.50mm, F.Cu at (119.4, 86.4)
- added J5: PWR, Connector_PinHeader_2.54mm:PinHeader_1x03_P2.54mm_Vertical, F.Cu at (101.6, 87.6)
- C1, C2, C3, C4, C5, C6, C7, C8: footprint Capacitor_THT:C_Disc_D12.5mm_W5.0mm_P10.00mm -> Capacitor_THT:C_Disc_D10.0mm_W2.5mm_P5.00mm
- moved C5 241.0 mm to (-111.5, 4.35)
- moved R22 241.0 mm to (-134.0, 50.4)
- moved R27 241.0 mm to (-147.3, 61.9)
- moved R31 241.0 mm to (-147.3, 57.9)
- moved R52 241.0 mm to (-134.0, 58.5)
- moved R62 241.0 mm to (-134.0, 62.5)
- moved R68 241.0 mm to (-147.3, 66.0)
- moved U7 241.0 mm to (-183.6, 3.15)
- moved C3 241.0 mm to (-151.1, 37.9)
- moved C4 241.0 mm to (-125.5, 10.9)
- moved C6 241.0 mm to (-125.5, 17.4)
- moved C7 241.0 mm to (-125.5, 4.35)
- moved C8 241.0 mm to (-151.1, 31.4)
- moved J2 241.0 mm to (-160.0, 30.4)
- moved J3 241.0 mm to (-195.7, 57.4)
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