File: hardware/vgagenerator.kicad_sch (KiCad schematic)
At the start: 90 parts, among them J1 VGA1, J2 VGA2, J3 VGA3, J4 VGA4, U1 Pico, U2 74HC374, U3 74HC374, U4 74HC374, U5 74HC374, U6 74HC374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

Commit message: Updated schematic
Parts:
- C1, C2, C3, C4, C5, C6, C7, C8: footprint (none) -> Capacitor_THT:C_Disc_D12.5mm_W5.0mm_P10.00mm
Changed lines of the file:
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@@
       (effects (font (size 1.27 1.27)) (justify left))
     )
-    (property "Footprint" "" (id 2) (at 33.9852 236.22 0)
+    (property "Footprint" "Capacitor_THT:C_Disc_D12.5mm_W5.0mm_P10.00mm" (id 2) (at 33.9852 236.22 0)
       (effects (font (size 1.27 1.27)) hide)
     )
@@
       (effects (font (size 1.27 1.27)) (justify left))
     )
-    (property "Footprint" "" (id 2) (at 72.0852 236.22 0)
+    (property "Footprint" "Capacitor_THT:C_Disc_D12.5mm_W5.0mm_P10.00mm" (id 2) (at 72.0852 236.22 0)
       (effects (font (size 1.27 1.27)) hide)
     )
@@
       (effects (font (size 1.27 1.27)) (justify left))
     )
-    (property "Footprint" "" (id 2) (at 110.1852 236.22 0)
+    (property "Footprint" "Capacitor_THT:C_Disc_D12.5mm_W5.0mm_P10.00mm" (id 2) (at 110.1852 236.22 0)
       (effects (font (size 1.27 1.27)) hide)
     )
@@
       (effects (font (size 1.27 1.27)) (justify left))
     )
-    (property "Footprint" "" (id 2) (at 59.3852 236.22 0)
+    (property "Footprint" "Capacitor_THT:C_Disc_D12.5mm_W5.0mm_P10.00mm" (id 2) (at 59.3852 236.22 0)
       (effects (font (size 1.27 1.27)) hide)
     )
@@
       (effects (font (size 1.27 1.27)) (justify left))
     )
-    (property "Footprint" "" (id 2) (at 84.7852 236.22 0)
+    (property "Footprint" "Capacitor_THT:C_Disc_D12.5mm_W5.0mm_P10.00mm" (id 2) (at 84.7852 236.22 0)
       (effects (font (size 1.27 1.27)) hide)
     )
@@
       (effects (font (size 1.27 1.27)) (justify left))
     )
-    (property "Footprint" "" (id 2) (at 97.4852 236.22 0)
+    (property "Footprint" "Capacitor_THT:C_Disc_D12.5mm_W5.0mm_P10.00mm" (id 2) (at 97.4852 236.22 0)
       (effects (font (size 1.27 1.27)) hide)
     )
@@
       (effects (font (size 1.27 1.27)) (justify left))
     )
-    (property "Footprint" "" (id 2) (at 46.6852 236.22 0)
+    (property "Footprint" "Capacitor_THT:C_Disc_D12.5mm_W5.0mm_P10.00mm" (id 2) (at 46.6852 236.22 0)
       (effects (font (size 1.27 1.27)) hide)
     )
@@
       (effects (font (size 1.27 1.27)) (justify left))
     )
-    (property "Footprint" "" (id 2) (at 21.2852 236.22 0)
+    (property "Footprint" "Capacitor_THT:C_Disc_D12.5mm_W5.0mm_P10.00mm" (id 2) (at 21.2852 236.22 0)
       (effects (font (size 1.27 1.27)) hide)
     )
@@
     )
     (path "/eee67514-f32f-4a4d-a6e5-63980cfec025"
-      (reference "C1") (unit 1) (value "100nF") (footprint "")
+      (reference "C1") (unit 1) (value "100nF") (footprint "Capacitor_THT:C_Disc_D12.5mm_W5.0mm_P10.00mm")
     )
     (path "/25772d3c-3662-40bd-8286-bb7869d35430"
-      (reference "C2") (unit 1) (value "100nF") (footprint "")
+      (reference "C2") (unit 1) (value "100nF") (footprint "Capacitor_THT:C_Disc_D12.5mm_W5.0mm_P10.00mm")
     )
     (path "/d4770399-802f-4512-b846-b240e0965432"
-      (reference "C3") (unit 1) (value "100nF") (footprint "")
+      (reference "C3") (unit 1) (value "100nF") (footprint "Capacitor_THT:C_Disc_D12.5mm_W5.0mm_P10.00mm")
     )
     (path "/5cd5ec75-54f0-462c-bd04-e83afdaef027"
-      (reference "C4") (unit 1) (value "100nF") (footprint "")
+      (reference "C4") (unit 1) (value "100nF") (footprint "Capacitor_THT:C_Disc_D12.5mm_W5.0mm_P10.00mm")
     )
     (path "/2ca17ea0-f952-4e98-9706-c5e0b793a49c"
-      (reference "C5") (unit 1) (value "100nF") (footprint "")
+      (reference "C5") (unit 1) (value "100nF") (footprint "Capacitor_THT:C_Disc_D12.5mm_W5.0mm_P10.00mm")
     )
     (path "/5d6fbce8-2a1c-44a3-a503-671e7a376491"
-      (reference "C6") (unit 1) (value "100nF") (footprint "")
+      (reference "C6") (unit 1) (value "100nF") (footprint "Capacitor_THT:C_Disc_D12.5mm_W5.0mm_P10.00mm")
     )
     (path "/6ffafaab-ac90-4a3d-914f-58e01a2425e2"
-      (reference "C7") (unit 1) (value "100nF") (footprint "")
+      (reference "C7") (unit 1) (value "100nF") (footprint "Capacitor_THT:C_Disc_D12.5mm_W5.0mm_P10.00mm")
     )
     (path "/54ac8b51-c308-4484-98bc-343374c4716e"
-      (reference "C8") (unit 1) (value "100nF") (footprint "")
+      (reference "C8") (unit 1) (value "100nF") (footprint "Capacitor_THT:C_Disc_D12.5mm_W5.0mm_P10.00mm")
     )
     (path "/5f0b9e5b-a1b9-4712-8208-0ffa8ec3159d"

Commit message: Updated schematics
Parts:
- added C9: 10uF x 10V, Capacitor_THT:C_Radial_D6.3mm_H11.0mm_P2.50mm, symbol Device:C_Polarized
- added J5: PWR, Connector_PinHeader_2.54mm:PinHeader_1x03_P2.54mm_Vertical, symbol Connector_Generic:Conn_01x03
- C1, C2, C3, C4, C5, C6, C7, C8: footprint Capacitor_THT:C_Disc_D12.5mm_W5.0mm_P10.00mm -> Capacitor_THT:C_Disc_D10.0mm_W2.5mm_P5.00mm
Connections:
- net +5V: now also C9.1, J5.2 (Pin_2)
- net GND: now also C9.2, J5.1 (Pin_1), J5.3 (Pin_3)
- no-connect marks 15 -> 18
